File: ESP_PLC.kicad_pcb (KiCad board)
At the start: 2 copper layers, 95 x 84 mm, 183 parts, among them J1 RJ45_Bel_SI-60062-F, J11 Screw_Terminal_01x06, J12 Screw_Terminal_01x03, J13 Screw_Terminal_01x02, J14 Screw_Terminal_01x02, J15 Screw_Terminal_01x02, J16 Screw_Terminal_01x02, J3 USB_C_Receptacle_USB2.0_14P, J4 Conn_01x06, J9 Screw_Terminal_01x06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

Commit message: development
Parts:
- removed R30, R31, R32, R33: ~400Ω, Resistor_SMD:R_1206_3216Metric
- moved D7 7.65 mm to (228.1, 111.0), turned to 45 degrees
- moved D9 1.06 mm to (171.3, 78.2)
- moved J14 0.80 mm to (160.4, 147.2)
- moved J16 0.80 mm to (194.1, 147.2)
- moved J13 0.80 mm to (143.7, 147.2)
- moved J15 0.80 mm to (177.2, 147.2)
- moved C13 0.51 mm to (224.3, 101.7)
- moved R9 0.40 mm to (223.6, 103.9)
Connections:
- J1 pad 12: +3.3V -> +3.3VA
- J1 pad 9: +3.3V -> +3.3VA
- K1 pad A1: Net-(K1-PadA1) -> VIN
- K2 pad A1: Net-(K2-PadA1) -> VIN
- K3 pad A1: Net-(K3-PadA1) -> VIN
- K4 pad A1: Net-(K4-PadA1) -> VIN
Routing:
- net +3.3VA: track 57.5 -> 126.0 mm, vias 6 -> 7
- net +3.3V: track 208.8 -> 152.5 mm, vias 13 -> 12
- net VIN: track 118.3 -> 138.2 mm
- net LINKLED: track 37.5 -> 29.0 mm
- net Net-(K1-PadA1): track 6.28 -> 0.00 mm
- net Net-(K2-PadA1): track 6.20 -> 0.00 mm
- net Net-(K3-PadA1): track 6.17 -> 0.00 mm
- net Net-(K4-PadA1): track 6.05 -> 0.00 mm
- net AGND: track 35.3 -> 37.0 mm
- net VTERM: track 55.9 -> 54.6 mm
- net ACTLED: track 31.3 -> 32.2 mm
- net GND: vias 60 -> 58
- net Earth: vias 29 -> 13
Other:
- board text added: "IO0"
- board text added: "RST"
- board text added: "VIN 4-32V"
- board text removed: "VIN 12-32V"
