File: IO.kicad_sch (KiCad schematic)
At the start: 154 parts, among them J1 RJ45_Bel_SI-60062-F, J11 Screw_Terminal_01x06, J12 Screw_Terminal_01x03, J13 Screw_Terminal_01x02, J14 Screw_Terminal_01x02, J15 Screw_Terminal_01x02, J16 Screw_Terminal_01x02, J4 Conn_01x06, J9 Screw_Terminal_01x06, K1 Relay_SPDT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

Commit message: development
Parts:
- removed R30, R31, R32, R33: ~400Ω, Resistor_SMD:R_1206_3216Metric, symbol Device:R_Small
Connections:
- net +3.3V: no longer J1.12, J1.9
- net +3.3VA: now also J1.12, J1.9
- net VIN: now also K1.A1, K2.A1, K3.A1, K4.A1
